Commit message: version 1.1

File: simple_robot.urdf (robot description, URDF)
Before this commit: robot simple_biped_with_even_larger_feet, 7 links, 6 joints
Links:
- link torso: mass 5.0 -> 1.5
Joints:
- joint left_ankle_joint: limit lower=-0.5 upper=0.5 effort=30 velocity=1.0 -> lower=-0.5 upper=0.5 effort=48 velocity=2.0
- joint left_hip_joint: limit lower=-1.57 upper=1.57 effort=50 velocity=1.0 -> lower=-1.57 upper=1.57 effort=80 velocity=2.0
- joint left_knee_joint: limit lower=0 upper=2.0 effort=50 velocity=1.0 -> lower=0 upper=2.0 effort=80 velocity=2.0
- joint right_ankle_joint: limit lower=-0.5 upper=0.5 effort=30 velocity=1.0 -> lower=-0.5 upper=0.5 effort=48 velocity=2.0
- joint right_hip_joint: limit lower=-1.57 upper=1.57 effort=50 velocity=1.0 -> lower=-1.57 upper=1.57 effort=80 velocity=2.0
- joint right_knee_joint: limit lower=0 upper=2.0 effort=50 velocity=1.0 -> lower=0 upper=2.0 effort=80 velocity=2.0

Commit message: version 1.2

File: simple_robot.urdf (robot description, URDF)
Before this commit: robot simple_biped_with_even_larger_feet, 7 links, 6 joints
Links:
- link left_foot: geometry collision box size=0.20 0.10 0.02; visual box size=0.20 0.10 0.02
- link right_foot: geometry collision box size=0.20 0.10 0.02; visual box size=0.20 0.10 0.02
- link torso: mass 1.5 -> 2.0; geometry collision box size=0.17 0.17 0.15; visual box size=0.17 0.17 0.15
